File: Hardware/bass_keyboard/bass_keyboard.kicad_pcb (KiCad board)
At the start: 2 copper layers, 186 parts

Commit message: Finishing layout, routing
Got all of the footprints where they need to be, created the pcb outline, and used Freerouting to route connections, doing some final connections by hand.
Parts:
- added J1: Conn_02x17_Top_Bottom, Connector_IDC:IDC-Header_2x17_P2.54mm_Vertical, B.Cu at (109.7, 228.6)
- added LS1: Speaker, Connector_Wire:SolderWire-2sqmm_1x02_P7.8mm_D2mm_OD3.9mm, F.Cu at (311.9, 106.4)
- D1, D10, D11, D12, D13, D14, D15, D16, D17, D18, D19, D2, D20, D21, D22, D23, D24, D25, D26, D27, D28, D29, D3, D30, D31, D32, D33, D34, D35, D36, D37, D38, D39, D4, D40, D41, D42, D43, D44, D45, D46, D47, D48, D49, D5, D50, D51, D52, D53, D54, D55, D56, D57, D58, D59, D6, D60, D61, D62, D63, D64, D65, D66, D67, D68, D69, D7, D70, D71, D72, D73, D74, D75, D76, D77, D78, D79, D8, D80, D81, D82, D83, D84, D85, D86, D87, D88, D89, D9, D90, D91: moved to B.Cu
- MX_down_half1: footprint Button_Switch_Keyboard:SW_Cherry_MX_1.00u_PCB -> Button_Switch_Keyboard:SW_Cherry_MX_1.50u_PCB
- MX_down_oct1, MX_func0: footprint Button_Switch_Keyboard:SW_Cherry_MX_1.00u_PCB -> Button_Switch_Keyboard:SW_Cherry_MX_2.00u_PCB
- MX_func11: footprint Button_Switch_Keyboard:SW_Cherry_MX_1.00u_PCB -> Button_Switch_Keyboard:SW_Cherry_MX_2.75u_PCB
- MX_func4: footprint Button_Switch_Keyboard:SW_Cherry_MX_1.00u_PCB -> Button_Switch_Keyboard:SW_Cherry_MX_6.25u_PCB
- MX_func8, MX_up_half1: footprint Button_Switch_Keyboard:SW_Cherry_MX_1.00u_PCB -> Button_Switch_Keyboard:SW_Cherry_MX_1.75u_PCB
- MX_maj_dom1: footprint Button_Switch_Keyboard:SW_Cherry_MX_1.00u_PCB -> Button_Switch_Keyboard:SW_Cherry_MX_1.25u_PCB
- MX_up_oct1: footprint Button_Switch_Keyboard:SW_Cherry_MX_1.00u_PCB -> Button_Switch_Keyboard:SW_Cherry_MX_2.25u_PCB
- moved MX_func2 432.7 mm to (113.7, 202.1)
- moved MX_Bn_min1 411.6 mm to (251.8, 144.9)
- moved MX_func3 410.3 mm to (132.7, 202.1)
- moved MX_Eb_dim1 409.3 mm to (108.9, 183.0)
- moved MX_maj_dom1 403.3 mm to (297.0, 164.0)
- moved MX_Gn_7 391.1 mm to (180.3, 164.0)
- moved MX_Fn_dim1 389.3 mm to (147.0, 183.0)
- moved MX_func4 388.6 mm to (151.8, 202.1)
- moved MX_Bb_7 376.5 mm to (123.2, 164.0)
- moved D79 373.7 mm to (61.1, 207.2), turned to 90 degrees
- moved MX_Ab_7 373.6 mm to (85.1, 164.0)
- moved MX_Gn_dim1 370.1 mm to (185.1, 183.0)
- moved MX_func5 367.8 mm to (170.8, 202.1)
- moved D66 361.3 mm to (58.7, 188.1), turned to 90 degrees
- moved MX_Cn_7 360.6 mm to (161.3, 164.0)
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Routing:
- net ROW0: track 0.00 -> 488.0 mm
- net ROW2: track 0.00 -> 449.9 mm, vias 0 -> 2
- net ROW1: track 0.00 -> 411.9 mm, vias 0 -> 2
- net ROW3: track 0.00 -> 411.6 mm, vias 0 -> 2
- net ROW5: track 0.00 -> 374.3 mm, vias 0 -> 4
- net COL11: track 0.00 -> 337.6 mm
- net COL12: track 0.00 -> 333.5 mm
- net Net-(J1-Pin_19): track 0.00 -> 331.0 mm, vias 0 -> 1
- net COL10: track 0.00 -> 327.3 mm
- net Net-(J1-Pin_20): track 0.00 -> 313.7 mm, vias 0 -> 2
- net ROW4: track 0.00 -> 301.9 mm, vias 0 -> 4
- net COL9: track 0.00 -> 291.5 mm, vias 0 -> 2
- net ROW6: track 0.00 -> 280.9 mm
- net COL8: track 0.00 -> 273.4 mm, vias 0 -> 2
- net COL7: track 0.00 -> 265.9 mm, vias 0 -> 1
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Other:
- board outline added: 291.3 x 154.8 mm
